File: src/USBSound.kicad_pcb (KiCad board)
At the start: 2 copper layers, 61 x 37.2 mm, 45 parts, among them J1 AudioJack4, J2 AudioJack4, J4 Mini-DIN-8, U1 CM108B, U2 USBLC6-2SC6, U3 AT3H7C-CuH-S

Commit message: Remove 10k attenuation resistor from potentiometers
Parts:
- removed R2, R9: 10k, Resistor_SMD:R_0805_2012Metric
- moved C10 11.0 mm to (158.8, 106.8), turned to 90 degrees
Connections:
- RV1 pad 3: Net-(R2-Pad1) -> /AFIN
- RV2 pad 1: Net-(R9-Pad2) -> Net-(C5-Pad1)
Routing:
- net Net-(R2-Pad1): track 4.06 -> 0.00 mm
- net /AFIN: track 30.5 -> 34.2 mm
- net Net-(R9-Pad2): track 3.71 -> 0.00 mm
- net Net-(C5-Pad1): track 6.49 -> 8.36 mm
- net GND: vias 94 -> 98
